Commit message: second commit

File: mec_mobile/mec_mobile_description/urdf/robots/robot_3d.urdf.xacro (robot description, xacro)
@@ -111,53 +111,3 @@
     <mu2>0.000002</mu2>
     </gazebo>
-  <!-- ros2_control: mô tả 4 bánh cho Gazebo + sau này HW thật -->
-  <ros2_control name="GazeboSimSystem" type="system">
-    <hardware>
-      <!-- Trong Gazebo dùng plugin này để nối với physics engine -->
-      <plugin>gz_ros2_control/GazeboSimSystem</plugin>
-    </hardware>
-    <!-- front_left -->
-    <joint name="front_left_wheel_joint">
-      <command_interface name="velocity">
-        <param name="min">-50.0</param>
-        <param name="max">50.0</param>
-      </command_interface>
-      <state_interface name="position"/>
-      <state_interface name="velocity"/>
-    </joint>
-    <!-- front_right -->
-    <joint name="front_right_wheel_joint">
-      <command_interface name="velocity">
-        <param name="min">-50.0</param>
-        <param name="max">50.0</param>
-      </command_interface>
-      <state_interface name="position"/>
-      <state_interface name="velocity"/>
-    </joint>
-    <!-- back_left -->
-    <joint name="back_left_wheel_joint">
-      <command_interface name="velocity">
-        <param name="min">-50.0</param>
-        <param name="max">50.0</param>
-      </command_interface>
-      <state_interface name="position"/>
-      <state_interface name="velocity"/>
-    </joint>
-    <!-- back_right -->
-    <joint name="back_right_wheel_joint">
-      <command_interface name="velocity">
-        <param name="min">-50.0</param>
-        <param name="max">50.0</param>
-      </command_interface>
-      <state_interface name="position"/>
-      <state_interface name="velocity"/>
-    </joint>
-  </ros2_control>
-    <gazebo>
-    <plugin
-      name="gz_ros2_control"
-      filename="gz_ros2_control-system">
-      <parameters>$(find mec_mobile_description)/config/mec_mobile_controllers.yaml</parameters>
-    </plugin>
-  </gazebo>
 </robot>
